Commit message: [#58] Modify urdf file for colllarm

File: robot/rospackages/src/colllarm/urdf/colllarm.urdf (robot description, URDF)
Before this commit: robot colllarm, 8 links, 6 joints
Joints:
- added joint finger1_joint: type prismatic, parent base_link, child finger1_link, origin xyz=0 0.018258 1.034 rpy=1.5708 0 0, axis 0 0 1, limit lower=-1.57 upper=1.57 effort=5 velocity=0.5
